File: VEXBridge.kicad_sch (KiCad schematic)
At the start: 28 parts, among them J1 4P4C, J3 Conn_01x05_Pin, U1 LM2596S-5, U2 MAX481E, U5 SN74LVC2G14DBV

Commit message: Fixed File Names
Used to be part of the BlueBox project :/
Other:
- title: BlueBox-PCB -> VEXBridge-PCB
Changed lines of the file:
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@@
 	(paper "A4")
 	(title_block
-		(title "BlueBox-PCB")
+		(title "VEXBridge-PCB")
 		(date "2024-11-25")
 		(rev "1.0")
@@
 		)
 		(instances
-			(project "BlueBox"
+			(project "VEXBridge"
 				(path "/75715a9c-a502-40d6-b270-e5c0bc6847fe"
 					(reference "R4")
@@
 		)
 		(instances
-			(project "BlueBox"
+			(project "VEXBridge"
 				(path "/75715a9c-a502-40d6-b270-e5c0bc6847fe"
 					(reference "R2")
@@
 		)
 		(instances
-			(project "BlueBox"
+			(project "VEXBridge"
 				(path "/75715a9c-a502-40d6-b270-e5c0bc6847fe"
 					(reference "H3")
@@
 		)
 		(instances
-			(project "BlueBox"
+			(project "VEXBridge"
 				(path "/75715a9c-a502-40d6-b270-e5c0bc6847fe"
 					(reference "#PWR09")
@@
 		)
 		(instances
-			(project "BlueBox"
+			(project "VEXBridge"
 				(path "/75715a9c-a502-40d6-b270-e5c0bc6847fe"
 					(reference "D3")
@@
 		)
 		(instances
-			(project "BlueBox"
+			(project "VEXBridge"
 				(path "/75715a9c-a502-40d6-b270-e5c0bc6847fe"
 					(reference "#PWR016")
@@
 		)
 		(instances
-			(project "BlueBox"
+			(project "VEXBridge"
 				(path "/75715a9c-a502-40d6-b270-e5c0bc6847fe"
 					(reference "C4")
@@
 		)
 		(instances
-			(project "BlueBox"
+			(project "VEXBridge"
 				(path "/75715a9c-a502-40d6-b270-e5c0bc6847fe"
 					(reference "#PWR012")
@@
 		)
 		(instances
-			(project "BlueBox"
+			(project "VEXBridge"
 				(path "/75715a9c-a502-40d6-b270-e5c0bc6847fe"
 					(reference "H2")
@@
 		)
 		(instances
-			(project "BlueBox"
+			(project "VEXBridge"
 				(path "/75715a9c-a502-40d6-b270-e5c0bc6847fe"
 					(reference "R3")
@@
 		)
 		(instances
-			(project "BlueBox"
+			(project "VEXBridge"
 				(path "/75715a9c-a502-40d6-b270-e5c0bc6847fe"
 					(reference "R7")
@@
 		)
 		(instances
-			(project "BlueBox"
+			(project "VEXBridge"
 				(path "/75715a9c-a502-40d6-b270-e5c0bc6847fe"
 					(reference "#PWR019")
@@
 		)
 		(instances
-			(project "BlueBox"
+			(project "VEXBridge"
 				(path "/75715a9c-a502-40d6-b270-e5c0bc6847fe"
 					(reference "H4")
@@
 		)
 		(instances
-			(project "BlueBox"
+			(project "VEXBridge"
 				(path "/75715a9c-a502-40d6-b270-e5c0bc6847fe"
 					(reference "D2")
@@
 		)
 		(instances
-			(project "BlueBox"
+			(project "VEXBridge"
 				(path "/75715a9c-a502-40d6-b270-e5c0bc6847fe"
 					(reference "R9")
@@
 		)
 		(instances
-			(project "BlueBox"
+			(project "VEXBridge"
 				(path "/75715a9c-a502-40d6-b270-e5c0bc6847fe"
 					(reference "R8")
@@
 		)
 		(instances
-			(project "BlueBox"
+			(project "VEXBridge"
 				(path "/75715a9c-a502-40d6-b270-e5c0bc6847fe"
 					(reference "C2")
@@
 		)
 		(instances
-			(project "BlueBox"
+			(project "VEXBridge"
 				(path "/75715a9c-a502-40d6-b270-e5c0bc6847fe"
 					(reference "#PWR011")
@@
 		)
 		(instances
-			(project "BlueBox"
+			(project "VEXBridge"
 				(path "/75715a9c-a502-40d6-b270-e5c0bc6847fe"
 					(reference "#PWR017")

Commit message: Increased Inductor Footprint
Parts:
- L1: footprint Inductor_SMD:L_Coilcraft_XxL4020 -> Inductor_SMD:L_Coilcraft_LPS4018
Changed lines of the file:
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@@
 			)
 		)
-		(property "Footprint" "Inductor_SMD:L_Coilcraft_XxL4020"
+		(property "Footprint" "Inductor_SMD:L_Coilcraft_LPS4018"
 			(at 100.33 100.33 0)
 			(effects
